Commit message: Arthur new configs

File: arthur/description.urdf (robot description, URDF)
Before this commit: robot arthur, 12 links, 11 joints
Joints:
- joint body_camera: origin xyz=0.15 0 0.25 rpy=0 0 0 -> xyz=0.15 0 0.25 rpy=0 -0.35 0

Commit message: Arthur Config

File: arthur/description.urdf (robot description, URDF)
Before this commit: robot arthur, 12 links, 11 joints
Links:
- removed link base_joint_link
- removed link yaw
Joints:
- removed joint pitch_base_joint
- removed joint roll_base_joint
- joint Eyes_Pitch: origin xyz=0.103 0 0.06 rpy=0 0 0 -> xyz=0.15 0 0.06 rpy=0 0 0
- joint blender_joint: origin xyz=0 0 0.62 rpy=0 0 0 -> xyz=0 0 0.6 rpy=0 0 0
- joint body_camera: origin xyz=0.15 0 0.25 rpy=0 0 0 -> xyz=0.15 0 0.25 rpy=0 -0.2 0
- joint roll_neck_joint: origin xyz=0.009 0 0.112 rpy=0 0 0 -> xyz=0.009 0 0.09 rpy=0 0 0
- joint yaw_joint: origin xyz=0 0 0 rpy=0 0 0 -> xyz=0 0 0.45 rpy=0 0 0; parent yaw -> body
